Commit message: controller fixed

File: ugv_description/urdf/bot.urdf.xacro (robot description, xacro)
@@ -28,4 +28,7 @@
     </inertial>
   </link>
+  <gazebo reference="base_link">
+    <material>Gazebo/DarkGrey</material>
+  </gazebo>
   <link name="wheel_front_right">
     <inertial>
@@ -104,4 +107,44 @@
     </collision>
   </link>
+  <gazebo reference="wheel_front_right">
+    <mu1>2.0</mu1>
+    <mu2>1.8</mu2>
+    <kp>200000.0</kp>
+    <kd>20.0</kd>
+    <minDepth>0.001</minDepth>
+    <maxVel>1</maxVel>
+    <fdir1>1 0 0</fdir1>
+    <material>Gazebo/Black</material>
+  </gazebo>
+  <gazebo reference="wheel_front_left">
+    <mu1>2.0</mu1>
+    <mu2>1.8</mu2>
+    <kp>200000.0</kp>
+    <kd>20.0</kd>
+    <minDepth>0.001</minDepth>
+    <maxVel>1</maxVel>
+    <fdir1>1 0 0</fdir1>
+    <material>Gazebo/Black</material>
+  </gazebo>
+  <gazebo reference="wheel_back_right">
+    <mu1>2.0</mu1>
+    <mu2>1.8</mu2>
+    <kp>200000.0</kp>
+    <kd>20.0</kd>
+    <minDepth>0.001</minDepth>
+    <maxVel>1</maxVel>
+    <fdir1>1 0 0</fdir1>
+    <material>Gazebo/Black</material>
+  </gazebo>
+  <gazebo reference="wheel_back_left">
+    <mu1>2.0</mu1>
+    <mu2>1.8</mu2>
+    <kp>200000.0</kp>
+    <kd>20.0</kd>
+    <minDepth>0.001</minDepth>
+    <maxVel>1</maxVel>
+    <fdir1>1 0 0</fdir1>
+    <material>Gazebo/Black</material>
+  </gazebo>
   <link name="rgb_camera">
     <inertial>
@@ -125,18 +168,6 @@
     </collision>
   </link>
-  <joint name="camera_joint" type="fixed">
-    <origin xyz="-0.85 0 0.0" rpy="0 0.0 3.14"/>
-    <parent link="base_link"/>
-    <child link="rgb_camera"/>
-    <axis xyz="0.0 0 0"/>
-  </joint>
-  <joint type="fixed" name="camera_optical_joint">
-    <origin xyz="0 0 0" rpy="-1.5707 0 -1.5707"/>
-    <child link="camera_link_optical"/>
-    <parent link="rgb_camera"/>
-  </joint>
-  <link name="camera_link_optical">
-  </link>
   <gazebo reference="rgb_camera">
+    <material>Gazebo/Blue</material>
     <sensor type="camera" name="camera">
       <always_on>1</always_on>
@@ -171,4 +202,17 @@
     </sensor>
   </gazebo>
+  <joint name="camera_joint" type="fixed">
+    <origin xyz="-0.85 0 0.0" rpy="0 0.0 3.14"/>
+    <parent link="base_link"/>
+    <child link="rgb_camera"/>
+    <axis xyz="0.0 0 0"/>
+  </joint>
+  <joint type="fixed" name="camera_optical_joint">
+    <origin xyz="0 0 0" rpy="-1.5707 0 -1.5707"/>
+    <child link="camera_link_optical"/>
+    <parent link="rgb_camera"/>
+  </joint>
+  <link name="camera_link_optical">
+  </link>
   <link name="laser_link">
     <inertial>
@@ -199,36 +243,30 @@
   </joint>
   <gazebo reference="laser_link">
-  <sensor type="ray" name="lidar_sensor">
-    <update_rate>50</update_rate>
-    <visualize>true</visualize>
-    <ray>
-      <scan>
-        <horizontal>
-          <samples>1800</samples>
-          <resolution>0.2</resolution>
-          <min_angle>-3.1415926</min_angle>
-          <max_angle>3.1415926</max_angle>
-        </horizontal>
-      </scan>
-      <range>
-        <min>0.3</min>
-        <max>100.0</max>
-        <resolution>0.001</resolution>
-      </range>
-    </ray>
-    <plugin name="gazebo_ros_laser" filename="libgazebo_ros_ray_sensor.so">
-      <topicName>/scan</topicName>
-      <frameName>laser_link</frameName>
-    </plugin>
-  </sensor>
-</gazebo>
-  <gazebo reference="lidar_base">
-    <material>Gazebo/DarkGrey</material>
-  </gazebo>
-  <gazebo reference="laser_link">
     <material>Gazebo/Black</material>
-  </gazebo>
-  <gazebo reference="lidar_dome">
-    <material>Gazebo/GreyTransparent</material>
+        <sensor name="laser" type="ray">
+            <pose> 0 0 0 0 0 0 </pose>
+            <visualize>false</visualize>
+            <update_rate>10</update_rate>
+            <ray>
+                <scan>
+                    <horizontal>
+                        <samples>360</samples>
+                        <min_angle>-3.14</min_angle>
+                        <max_angle>3.14</max_angle>
+                    </horizontal>
+                </scan>
+                <range>
+                    <min>0.3</min>
+                    <max>12</max>
+                </range>
+            </ray>
+            <plugin name="laser_controller" filename="libgazebo_ros_ray_sensor.so">
+                <ros>
+                    <argument>~/out:=scan</argument>
+                </ros>
+                <output_type>sensor_msgs/LaserScan</output_type>
+                <frame_name>laser_link</frame_name>
+            </plugin>
+        </sensor>
   </gazebo>
   <link name="navsat_link">
@@ -292,62 +330,4 @@
     <axis xyz="0.0 0.0 1.0"/>
   </joint>
-  <gazebo reference="wheel_front_right">
-    <mu1>2.0</mu1>
-    <mu2>1.8</mu2>
-    <kp>200000.0</kp>
-    <kd>20.0</kd>
-    <minDepth>0.001</minDepth>
-    <maxVel>1</maxVel>
-    <fdir1>1 0 0</fdir1>
-  </gazebo>
-  <gazebo reference="wheel_front_left">
-    <mu1>2.0</mu1>
-    <mu2>1.8</mu2>
-    <kp>200000.0</kp>
-    <kd>20.0</kd>
-    <minDepth>0.001</minDepth>
-    <maxVel>1</maxVel>
-    <fdir1>1 0 0</fdir1>
-  </gazebo>
-  <gazebo reference="wheel_back_right">
-    <mu1>2.0</mu1>
-    <mu2>1.8</mu2>
-    <kp>200000.0</kp>
-    <kd>20.0</kd>
-    <minDepth>0.001</minDepth>
-    <maxVel>1</maxVel>
-    <fdir1>1 0 0</fdir1>
-  </gazebo>
-  <gazebo reference="wheel_back_left">
-    <mu1>2.0</mu1>
-    <mu2>1.8</mu2>
-    <kp>200000.0</kp>
-    <kd>20.0</kd>
-    <minDepth>0.001</minDepth>
-    <maxVel>1</maxVel>
-    <fdir1>1 0 0</fdir1>
-  </gazebo>
-<gazebo>
-  <plugin name="differential_drive_controller" filename="libgazebo_ros_diff_drive.so">
-    <left_joint>wheel_front_left_joint</left_joint>
-    <right_joint>wheel_front_right_joint</right_joint>
-    <wheel_separation>1.4</wheel_separation>
-    <wheel_diameter>0.56</wheel_diameter>
-    <wheel_acceleration>1.0</wheel_acceleration>
-    <wheel_torque>20</wheel_torque>
-    <max_wheel_torque>20</max_wheel_torque>
-    <command_topic>cmd_vel</command_topic>
-    <odometry_topic>odom</odometry_topic>
-    <odometry_frame>odom</odometry_frame>
-    <robot_base_frame>base_footprint</robot_base_frame>
-    <publish_odom>true</publish_odom>
-    <publish_wheel_tf>true</publish_wheel_tf>
-    <publish_odom_tf>true</publish_odom_tf>
-    <publish_wheel_joint_state>true</publish_wheel_joint_state>
-    <update_rate>50.0</update_rate>
-    <legacy_mode>false</legacy_mode>
-    <rosDebugLevel>Debug</rosDebugLevel>
-  </plugin>
-</gazebo>
   <link name="front_skid_plate">
     <inertial>

File: ugv_description/urdf/bot_ros2_control.xacro (robot description, xacro)
@@ -2,11 +2,7 @@
 <robot xmlns:xacro="http://www.ros.org/wiki/xacro" name="bot">
     <ros2_control name="RobotSystem" type="system">
-        <!-- ros2_control Gazebo -->
-        <!-- ROS 2 Humble -->
         <hardware>
-            <plugin>ign_ros2_control/IgnitionSystem</plugin>
+            <plugin>gazebo_ros2_control/GazeboSystem</plugin>
         </hardware>
-        <!-- ros2_control Common Interfaces -->
-        <!-- Front right wheel -->
         <joint name="wheel_front_right_joint">
             <command_interface name="velocity">
@@ -17,5 +13,4 @@
             <state_interface name="velocity" />
         </joint>
-        <!-- Front left wheel -->
         <joint name="wheel_front_left_joint">
             <command_interface name="velocity">
@@ -26,5 +21,4 @@
             <state_interface name="velocity" />
         </joint>
-        <!-- Back right wheel -->
         <joint name="wheel_back_right_joint">
             <command_interface name="velocity">
@@ -35,5 +29,4 @@
             <state_interface name="velocity" />
         </joint>
-        <!-- Back left wheel -->
         <joint name="wheel_back_left_joint">
             <command_interface name="velocity">
@@ -45,3 +38,11 @@
         </joint>
     </ros2_control>
+    <gazebo>
+        <plugin name="gazebo_ros2_control" filename="libgazebo_ros2_control.so">
+            <parameters>$(find ugv_description)/config/ugv_controller.yaml</parameters>
+            <ros>
+                <namespace>/</namespace>
+            </ros>
+        </plugin>
+    </gazebo>
 </robot>
